File: doc/Chassis2.kicad_sch (KiCad schematic)
At the start: 17 parts, among them M1 GM37-520-R, M2 GM37-520-R, M3 GM37-520-R, M4 GM37-520-R, U1 STM32F411CEUx

Commit message: update readme
Parts:
- added R2, R3: R, symbol Device:R
Connections:
- net GND1: now also R2.2, R3.2
- net at S1.5 (SCL), S2.5 (SCL), U1.45 (PB8): now also S1.6 (SDA), S2.6 (SDA), U1.46 (PB9), R2.1, R3.1
Changed lines of the file:
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@@
   (junction (at 199.39 53.34) (diameter 0) (color 0 0 0 0)
   )
+  (junction (at 256.54 99.06) (diameter 0) (color 0 0 0 0)
+  )
   (junction (at 64.77 68.58) (diameter 0) (color 0 0 0 0)
   )
+  (junction (at 262.89 101.6) (diameter 0) (color 0 0 0 0)
+  )
   (junction (at 59.69 142.24) (diameter 0) (color 0 0 0 0)
   )
@@
   (junction (at 223.52 97.79) (diameter 0) (color 0 0 0 0)
   )
+  (junction (at 262.89 109.22) (diameter 0) (color 0 0 0 0)
+  )
   (junction (at 215.9 100.33) (diameter 0) (color 0 0 0 0)
   )
@@
   (junction (at 64.77 77.47) (diameter 0) (color 0 0 0 0)
   )
+  (junction (at 251.46 100.33) (diameter 0) (color 0 0 0 0)
+  )
   (junction (at 67.31 50.8) (diameter 0) (color 0 0 0 0)
   )
@@
   (junction (at 213.36 143.51) (diameter 0) (color 0 0 0 0)
   )
+  (junction (at 254 101.6) (diameter 0) (color 0 0 0 0)
+  )
   (junction (at 218.44 101.6) (diameter 0) (color 0 0 0 0)
   )
@@
     (stroke (width 0) (type default) (color 0 0 0 0))
   )
+  (wire (pts (xy 251.46 100.33) (xy 262.89 100.33))
+    (stroke (width 0) (type default) (color 0 0 0 0))
+  )
   (wire (pts (xy 241.3 44.45) (xy 278.13 44.45))
     (stroke (width 0) (type default) (color 0 0 0 0))
@@
     (stroke (width 0) (type default) (color 0 0 0 0))
   )
+  (wire (pts (xy 262.89 101.6) (xy 273.05 101.6))
+    (stroke (width 0) (type default) (color 0 0 0 0))
+  )
   (wire (pts (xy 255.27 59.69) (xy 264.16 59.69))
     (stroke (width 0) (type default) (color 0 0 0 0))
@@
     (stroke (width 0) (type default) (color 0 0 0 0))
   )
+  (wire (pts (xy 256.54 99.06) (xy 256.54 109.22))
+    (stroke (width 0) (type default) (color 0 0 0 0))
+  )
   (wire (pts (xy 128.27 45.72) (xy 97.79 45.72))
     (stroke (width 0) (type default) (color 0 0 0 0))
@@
     (stroke (width 0) (type default) (color 0 0 0 0))
   )
+  (wire (pts (xy 254 101.6) (xy 262.89 101.6))
+    (stroke (width 0) (type default) (color 0 0 0 0))
+  )
   (wire (pts (xy 102.87 53.34) (xy 102.87 147.32))
     (stroke (width 0) (type default) (color 0 0 0 0))
@@
     (stroke (width 0) (type default) (color 0 0 0 0))
   )
+  (wire (pts (xy 262.89 109.22) (xy 273.05 109.22))
+    (stroke (width 0) (type default) (color 0 0 0 0))
+  )
   (wire (pts (xy 97.79 157.48) (xy 97.79 162.56))
     (stroke (width 0) (type default) (color 0 0 0 0))
@@
     (stroke (width 0) (type default) (color 0 0 0 0))
   )
+  (wire (pts (xy 256.54 109.22) (xy 262.89 109.22))
+    (stroke (width 0) (type default) (color 0 0 0 0))
+  )
   (wire (pts (xy 74.93 58.42) (xy 48.26 58.42))
     (stroke (width 0) (type default) (color 0 0 0 0))
@@
   )
   (wire (pts (xy 123.19 132.08) (xy 204.47 132.08))
+    (stroke (width 0) (type default) (color 0 0 0 0))
+  )
+  (wire (pts (xy 262.89 100.33) (xy 262.89 101.6))
     (stroke (width 0) (type default) (color 0 0 0 0))
   )
@@
     (pin "2")
   )
+  (symbol (lib_id "Device:R") (at 273.05 105.41 0) (unit 1)
+    (in_bom yes) (on_board yes) (fields_autoplaced)
+    (property "Reference" "R3" (id 0) (at 275.59 104.1399 0)
+      (effects (font (size 1.27 1.27)) (justify left))
+    )
+    (property "Value" "R" (id 1) (at 275.59 106.6799 0)
+      (effects (font (size 1.27 1.27)) (justify left))
+    )
+    (property "Footprint" "" (id 2) (at 271.272 105.41 90)
+      (effects (font (size 1.27 1.27)) hide)
+    )
+    (property "Datasheet" "~" (id 3) (at 273.05 105.41 0)
+      (effects (font (size 1.27 1.27)) hide)
+    )
+    (pin "1")
+    (pin "2")
+  )
   (symbol (lib_id "power:+5V") (at 59.69 22.86 0) (unit 1)
     (in_bom yes) (on_board yes) (fields_autoplaced)
@@
     )
     (pin "1")
+  )
+  (symbol (lib_id "Device:R") (at 262.89 105.41 0) (unit 1)
+    (in_bom yes) (on_board yes) (fields_autoplaced)
+    (property "Reference" "R2" (id 0) (at 265.43 104.1399 0)
+      (effects (font (size 1.27 1.27)) (justify left))
+    )
+    (property "Value" "R" (id 1) (at 265.43 106.6799 0)
+      (effects (font (size 1.27 1.27)) (justify left))
+    )
+    (property "Footprint" "" (id 2) (at 261.112 105.41 90)
+      (effects (font (size 1.27 1.27)) hide)
+    )
+    (property "Datasheet" "~" (id 3) (at 262.89 105.41 0)
+      (effects (font (size 1.27 1.27)) hide)
+    )
+    (pin "1")
+    (pin "2")
   )
   (symbol (lib_id "Device:Battery_Cell") (at 269.24 59.69 90) (unit 1)
@@
       (reference "R1") (unit 1) (value "R") (footprint "")
     )
+    (path "/27676708-2e01-41d9-8f7a-5ff06226243e"
+      (reference "R2") (unit 1) (value "R") (footprint "")
+    )
+    (path "/1654fb5f-aaba-4791-8001-45a4ce8b7bd9"
+      (reference "R3") (unit 1) (value "R") (footprint "")
+    )
     (path "/b9373311-7733-43ae-921f-cc9052de9140"
